File: DumbFCC.kicad_pcb (KiCad board)
At the start: 6 copper layers, 0 parts

Commit message: First draft of schematic
Parts:
- added BZ400: Buzzer, AI-1027-TWT-3V-R:XDCR_AI-1027-TWT-3V-R, F.Cu at (165.4, 72.0)
- added C100: 470n, Capacitor_SMD:C_0805_2012Metric, F.Cu at (178.5, 96.0)
- added C101: 470n, Capacitor_SMD:C_0805_2012Metric, F.Cu at (175.0, 96.0)
- added C200: 10u, Capacitor_SMD:CP_Elec_4x5.7, F.Cu at (141.5, 84.0)
- added C201: 100n, Capacitor_SMD:C_0805_2012Metric, F.Cu at (157.5, 76.5)
- added C202: 100n, Capacitor_SMD:C_0805_2012Metric, F.Cu at (163.5, 87.5)
- added C203: 100n, Capacitor_SMD:C_0805_2012Metric, F.Cu at (158.5, 92.5)
- added C204: 100n, Capacitor_SMD:C_0805_2012Metric, F.Cu at (151.5, 92.5)
- added C205: 100n, Capacitor_SMD:C_0805_2012Metric, F.Cu at (146.5, 82.5)
- added C207: 10p, Capacitor_SMD:C_0805_2012Metric, F.Cu at (142.2, 90.2)
- added C208: 10p, Capacitor_SMD:C_0805_2012Metric, F.Cu at (146.2, 94.2)
- added C300: 100n, Capacitor_SMD:C_0805_2012Metric, F.Cu at (133.5, 79.0)
- added C303: 220n, Capacitor_SMD:C_0805_2012Metric, F.Cu at (130.7, 81.3)
- added C304: 100n, Capacitor_SMD:C_0805_2012Metric, F.Cu at (131.0, 87.5)
- added C305: 100n, Capacitor_SMD:C_0805_2012Metric, F.Cu at (133.8, 87.0)
- added C306: 100n, Capacitor_SMD:C_0805_2012Metric, F.Cu at (122.9, 84.5)
- added C307: 10u, Capacitor_SMD:CP_Elec_4x5.7, F.Cu at (135.0, 71.0)
- added C308: 100n, Capacitor_SMD:C_0805_2012Metric, F.Cu at (134.9, 76.0)
- added C400: 100n, Capacitor_SMD:C_0805_2012Metric, B.Cu at (135.5, 95.3)
- added C401: 100n, Capacitor_SMD:C_0805_2012Metric, F.Cu at (152.5, 101.4)
- added C500: 100n, Capacitor_SMD:C_0805_2012Metric, B.Cu at (178.0, 84.5)
- added C501: 100n, Capacitor_SMD:C_0805_2012Metric, B.Cu at (174.0, 89.5)
- added D100: PWR, LED_SMD:LED_0805_2012Metric, F.Cu at (171.5, 92.0)
- added D400: FLT, LED_SMD:LED_0805_2012Metric, F.Cu at (163.5, 103.6)
- added D401: DBG, LED_SMD:LED_0805_2012Metric, F.Cu at (167.0, 103.6)
- added D402: VER, LED_SMD:LED_0805_2012Metric, F.Cu at (170.5, 103.6)
- added D403: SBY, LED_SMD:LED_0805_2012Metric, F.Cu at (174.0, 103.6)
- added D404: ERR, LED_SMD:LED_0805_2012Metric, F.Cu at (160.0, 103.6)
- added D500: TVS, Diode_SMD:D_SOD-323F, F.Cu at (172.6, 79.5)
- added D501: TVS, Diode_SMD:D_SOD-323F, F.Cu at (172.6, 76.2)
- added D502: D_Schottky, Diode_SMD:D_0805_2012Metric, F.Cu at (176.0, 85.0)
- added FB500: FerriteBead, Inductor_SMD:L_0805_2012Metric, F.Cu at (180.0, 85.0)
- added H200: M3_Pad, MountingHole:MountingHole_3.2mm_M3_Pad_TopBottom, F.Cu at (120.0, 65.0)
- added H201: M3_Pad, MountingHole:MountingHole_3.2mm_M3_Pad_TopBottom, F.Cu at (180.0, 65.0)
- added H202: M3_Pad, MountingHole:MountingHole_3.2mm_M3_Pad_TopBottom, F.Cu at (119.5, 105.0)
- added H203: M3_Pad, MountingHole:MountingHole_3.2mm_M3_Pad_TopBottom, F.Cu at (180.0, 105.5)
- added J100: 5V Input, Connector_PinHeader_2.54mm:PinHeader_1x02_P2.54mm_Vertical, F.Cu at (183.0, 92.3)
- added J300: Distance Sensor, Connector_PinHeader_2.54mm:PinHeader_1x04_P2.54mm_Vertical, F.Cu at (149.0, 108.2)
- added J402: SD port, 5027740891:MOLEX_5027740891, B.Cu at (124.0, 89.0)
- added J500: Debug, Connector_PinHeader_2.54mm:PinHeader_1x04_P2.54mm_Vertical, F.Cu at (139.9, 61.8)
- added J501: UART, Connector_PinHeader_2.54mm:PinHeader_1x04_P2.54mm_Vertical, F.Cu at (136.0, 108.2)
- added J502: I2C, Connector_PinHeader_2.54mm:PinHeader_1x04_P2.54mm_Vertical, F.Cu at (163.9, 61.8)
- added J503: CAN port, Connector_PinHeader_2.54mm:PinHeader_1x02_P2.54mm_Vertical, F.Cu at (183.0, 96.0)
- added J504: Motor, Connector_PinHeader_2.54mm:PinHeader_2x03_P2.54mm_Vertical, F.Cu at (153.0, 64.3)
- added J505: Gimbal, Connector_PinHeader_2.54mm:PinHeader_2x03_P2.54mm_Vertical, F.Cu at (128.5, 64.3)
- added J506: USB C, 2171790001_MOL:2171790001_MOL, F.Cu at (182.0, 78.0)
- added JP200: Boot, TestPoint:TestPoint_2Pads_Pitch2.54mm_Drill0.8mm, F.Cu at (151.6, 74.3)
- added JP300: SD0, Jumper:SolderJumper-2_P1.3mm_Open_TrianglePad1.0x1.5mm, F.Cu at (130.5, 95.5)
- added JP302: SD0, Jumper:SolderJumper-2_P1.3mm_Open_TrianglePad1.0x1.5mm, F.Cu at (126.0, 95.5)
- added R100: 330, Resistor_SMD:R_0805_2012Metric, F.Cu at (171.5, 96.0)
- added R200: 620, Resistor_SMD:R_0805_2012Metric, F.Cu at (147.7, 90.2)
- added R201: 10k, Resistor_SMD:R_0805_2012Metric, F.Cu at (152.9, 71.9)
- added R300: 10k, Resistor_SMD:R_0805_2012Metric, F.Cu at (130.5, 92.0)
- added R302: 10k, Resistor_SMD:R_0805_2012Metric, F.Cu at (126.0, 92.0)
- added R303: 10k, Resistor_SMD:R_0805_2012Metric, F.Cu at (148.0, 76.0)
- added R304: 10k, Resistor_SMD:R_0805_2012Metric, F.Cu at (145.5, 78.5)
- added R400: 10k, Resistor_SMD:R_0805_2012Metric, F.Cu at (136.0, 102.8)
- added R401: 10k, Resistor_SMD:R_0805_2012Metric, F.Cu at (136.0, 98.2)
- added R402: 330, Resistor_SMD:R_0805_2012Metric, F.Cu at (163.5, 107.3)
- added R403: 330, Resistor_SMD:R_0805_2012Metric, F.Cu at (167.0, 107.3)
- added R404: 330, Resistor_SMD:R_0805_2012Metric, F.Cu at (170.5, 107.3)
- added R405: 330, Resistor_SMD:R_0805_2012Metric, F.Cu at (174.0, 107.3)
- added R406: 330, Resistor_SMD:R_0805_2012Metric, F.Cu at (160.0, 107.3)
- added R500: 10k, Resistor_SMD:R_0805_2012Metric, F.Cu at (167.4, 65.8)
- added R501: 10k, Resistor_SMD:R_0805_2012Metric, F.Cu at (162.9, 65.8)
- added R502: 120, Resistor_SMD:R_0805_2012Metric, B.Cu at (177.9, 96.3)
- added R503: 5k1, Resistor_SMD:R_0805_2012Metric, F.Cu at (175.6, 80.2)
- added R504: 5k1, Resistor_SMD:R_0805_2012Metric, F.Cu at (175.5, 75.3)
- added SW400: Mode Switch, DS04-254-1-02BK-SMT:SW_DS04-254-1-02BK-SMT, F.Cu at (129.0, 100.5)
- added SW401: Reset, DTS-32N-V-B:DTS32NVB, F.Cu at (149.2, 97.4)
- added TP300: SDA, TestPoint:TestPoint_Pad_D1.5mm, F.Cu at (142.0, 72.5)
- added TP301: SCL, TestPoint:TestPoint_Pad_D1.5mm, F.Cu at (142.0, 76.0)
- added U100: ADP3330ARTZ3.3-RL7, Package_TO_SOT_SMD:SOT-23-6, F.Cu at (177.5, 92.0)
- added U200: STM32H573RIT6, Package_QFP:LQFP-64_10x10mm_P0.5mm, F.Cu at (155.0, 85.0)
- added U300: LIS2MDL, Package_LGA:LGA-12_2x2mm_P0.5mm, F.Cu at (131.0, 78.5)
- added U301: LSM6DSL, Package_LGA:LGA-14_3x2.5mm_P0.5mm_LayoutBorder3x4y, F.Cu at (131.0, 85.0)
- added U302: MS5607-02BA, Package_LGA:LGA-8_3x5mm_P1.25mm, F.Cu at (126.0, 85.5)
- added U400: AT25DF321A-SH-T, Package_SO:SOIC-8_3.9x4.9mm_P1.27mm, B.Cu at (137.0, 90.3)
- added U500: MCP2562T-E_SN, Package_SO:SOIC-8_5.3x5.3mm_P1.27mm, B.Cu at (178.0, 90.5)
- added Y200: 25MHz, Crystal:Crystal_SMD_Abracon_ABM8G-4Pin_3.2x2.5mm, F.Cu at (144.2, 92.2)
Routing:
- net +3V3: track 0.00 -> 335.6 mm, vias 0 -> 6
- net +5V: track 0.00 -> 143.9 mm, vias 0 -> 1
- net /Project Architecture/MCU/SPI_MISO: track 0.00 -> 50.0 mm, vias 0 -> 1
- net /Project Architecture/Connections/NRST: track 0.00 -> 48.4 mm, vias 0 -> 1
- net /Project Architecture/MCU/I2C_SENS_SDA: track 0.00 -> 46.4 mm, vias 0 -> 3
- net /Project Architecture/MCU/I2C_SENS_SCL: track 0.00 -> 44.7 mm, vias 0 -> 3
- net /Project Architecture/MCU/IMU_INT_1: track 0.00 -> 41.7 mm, vias 0 -> 2
- net /Project Architecture/Connections/GIMB_ROLL: track 0.00 -> 37.6 mm, vias 0 -> 1
- net /Project Architecture/MCU/SPI_SCK: track 0.00 -> 37.2 mm, vias 0 -> 1
- net /Project Architecture/Connections/UART_TX: track 0.00 -> 33.7 mm, vias 0 -> 1
- net /Project Architecture/MCU/TRIG: track 0.00 -> 33.4 mm
- net /Project Architecture/MCU/SPI_MOSI: track 0.00 -> 32.5 mm, vias 0 -> 1
- net /Project Architecture/Connections/UART_RX: track 0.00 -> 32.3 mm, vias 0 -> 1
- net /Project Architecture/MCU/ECHO: track 0.00 -> 32.0 mm
- net /Project Architecture/Connections/GIMB_PITCH: track 0.00 -> 31.9 mm, vias 0 -> 1
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- added copper zone on B.Cu, net +3V3
- added copper zone on F.Cu, net +3V3
- added copper zone on F.Cu, net +5V
- added copper zone on B.Cu, net GND
- added copper zone on F.Cu, net GND
- added copper zone on In1.Cu, net GND
- added copper zone on In2.Cu, net GND
Other:
- board outline added: 70 x 50 mm
- copper layers 6 -> 4
- rule pad_to_mask_clearance: 0.05 -> 0.1
- board text added: "+"
- board text added: "1"
- board text added: "2"
- board text added: "3V3"
- board text added: "4 x M3"
- board text added: "5V"
- board text added: "ADP 2025/26"
- board text added: "ALT"
- board text added: "BARO"
- board text added: "BOOT"
- board text added: "CAN"
- board text added: "DBG"
- board text added: "DEBUG"
- board text added: "DUMB FCC"
- board text added: "ECHO"
- board text added: "ERR"
- board text added: "FLT"
- board text added: "GIMBAL"
- board text added: "GND"
- board text added: "H"
- board text added: "I2C"
- board text added: "IMU"
- board text added: "L"
- board text added: "MOTOR"
- board text added: "NRST"
- board text added: "RESET"
- board text added: "RX"
- board text added: "Rev ${REVISION} ${RELEASE_DATE_NUM} Curtis Dickson"
- board text added: "SBY"
- board text added: "SCL"
- board text added: "SD"
- board text added: "SDA"
- board text added: "SIG"
- board text added: "SWCLK"
- board text added: "SWDIO"
- board text added: "TRIG"
- board text added: "TX"
- board text added: "UART"
- board text added: "VER"
- board text added: "x"
- board text added: "y"
- board text added: "z"
- board text added: "Φ"
- board text added: "θ"
- board text removed: "30°"
- board text removed: "3× 120°"
