File: Project Architecture.kicad_sch (KiCad schematic)
At the start: 0 parts

Commit message: First draft of schematic
Other:
- removed sheet Section A - Title A
- removed sheet Section B - Title B
- added sheet Connections (Connections.kicad_sch)
- added sheet MCU (MCU.kicad_sch)
- added sheet Peripherals (Peripherals.kicad_sch)
- added sheet Power (Power.kicad_sch)
- added sheet Sensors (Sensors.kicad_sch)
- note added: "Page 6"
- note added: "Page 7"
- note added: "Page 8"
